File: PCBs/Breakout Board/AERIS-Nano Breakout Board.kicad_pcb (KiCad board)
At the start: 2 copper layers, 42.5 x 35 mm, 9 parts, among them J1 Conn_01x04_Pin, J2 Conn_01x04_Pin, J3 Conn_01x02_Socket, Q1 2N2222, U1 ESP32C3

Commit message: Update PCB
Other:
- board text added: "1KΩ"
- board text removed: "1K"
Changed lines of the file:
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@@
 		)
 	)
-	(gr_text "1K"
+	(gr_text "1KΩ\n"
 		(at 183.5 102 0)
 		(layer "B.SilkS")
