File: PCBs/Breakout Board/AERIS-Nano Breakout Board.kicad_pcb (KiCad board)
At the start: 2 copper layers, 42.5 x 35 mm, 9 parts, among them J1 Conn_01x04_Pin, J2 Conn_01x04_Pin, J3 Conn_01x02_Socket, Q1 2N2222, U1 ESP32C3

Commit message: PCB V2
Parts:
- added DC: DC Jumper, Jumper:SolderJumper-2_P1.3mm_Open_RoundedPad1.0x1.5mm, F.Cu at (177.5, 95.0)
- moved R1 7.08 mm to (186.8, 102.5), turned to 90 degrees
- moved Q1 1.70 mm to (183.3, 97.5), turned to 180 degrees
- moved REF** 0.83 mm to (179.2, 107.2)
Routing:
- net /PWM: track 28.6 -> 34.1 mm
- net Net-(Q1-B): track 8.93 -> 7.04 mm
Other:
- board text added: "+5V DC"
- board text added: "AERIS-N V2"
- board text removed: "V1.0"
