File: PCBs/Breakout Board/AERIS-Nano Breakout Board.kicad_sch (KiCad schematic)
At the start: 6 parts, among them J1 Conn_01x04_Pin, J2 Conn_01x04_Pin, J3 Conn_01x02_Socket, Q1 2N2222, U1 ESP32C3

Commit message: PCB V2
Parts:
- added JP1: DC Jumper, Jumper:SolderJumper-2_P1.3mm_Open_RoundedPad1.0x1.5mm, symbol Jumper:Jumper_2_Open
- U1: value ESP32C3 -> ESP32-C3/C6
Connections:
- net GND: now also JP1.2 (B)
- net at J3.2 (Pin_2), Q1.3 (C): now also JP1.1 (A)
Other:
- note added: "XIAO ESP32-C3/C6"
- note removed: "XIAO ESP32C3"
- moved on the sheet: J1, J2
